File: hardware/rc-xbox-controller.kicad_sch (KiCad schematic)
At the start: 0 parts

Commit message: Add KiCad wiring schematic with all components
Parts:
- added C1: C, symbol Device:C
- added D1: LED, symbol Device:LED
- added M1, M2: Motor_DC, symbol Motor:Motor_DC
- added RV1: R_Potentiometer, symbol Device:R_Potentiometer
- added U1: ESP32-WROOM-32, RF_Module:ESP32-WROOM-32, symbol RF_Module:ESP32-WROOM-32
- added U2: TB6612FNG, Package_SO:SSOP-24_5.3x8.2mm_P0.65mm, symbol Driver_Motor:TB6612FNG
Connections:
- new net: D1.2 (A), U1.16 (IO13)
- new net: M2.1 (+), U2.1 (AO1), U2.2 (AO1)
- new net: U2.10 (PGND2), U2.9 (PGND2)
- new net: M1.1 (+), U2.11 (BO1), U2.12 (BO1)
- new net: U1.14 (IO12), U1.8 (IO32), U2.15 (PWMB), U2.23 (PWMA)
- new net: U1.13 (IO14), U2.16 (BIN2)
- new net: U1.12 (IO27), U2.17 (BIN1)
- new net: U1.11 (IO26), U2.19 (STBY)
- new net: U1.10 (IO25), U2.21 (AIN1)
- new net: U1.9 (IO33), U2.22 (AIN2)
- new net: U2.3 (PGND1), U2.4 (PGND1)
- new net: M2.2 (-), U2.5 (AO2), U2.6 (AO2)
- new net: M1.2 (-), U2.7 (BO2), U2.8 (BO2)
- new net: C1.1, RV1.2, U1.6 (IO34)
- new net +3.3V: C1.2, D1.1 (K), RV1.1, RV1.3, U1.1 (GND), U1.15 (GND), U1.2 (VDD), U1.38 (GND), U1.39 (GND)
- new net +5V: U2.20 (VCC)
Other:
- note added: "Head Lights"
- note added: "Rear motor"
- note added: "Steering Motor"

Commit message: Updated schematic: ERC clean, re-exported SVG + PDF
Parts:
- added R1: 220, symbol Device:R
- C1: value C -> 100nF
Connections:
- net +3.3V: no longer C1.2, D1.1 (K), RV1.3, U1.1 (GND), U1.15 (GND), U1.38 (GND), U1.39 (GND)
- net at D1.2 (A): now also R1.2; no longer U1.16 (IO13)
- net BIN2: now reaches U1.13 (IO14)
- net BIN2: no longer U2.16 (BIN2)
- net BIN1: now reaches U1.12 (IO27)
- net BIN1: no longer U2.17 (BIN1)
- net GND: now reaches U2.18 (GND)
- net GND: now also C1.2, D1.1 (K), RV1.3, U1.1 (GND), U1.15 (GND), U1.38 (GND), U1.39 (GND)
- net IO26: now reaches U2.19 (STBY)
- net IO26: no longer U1.11 (IO26)
- net AIN1: now reaches U1.10 (IO25)
- net AIN1: no longer U2.21 (AIN1)
- net AIN2: now reaches U1.9 (IO33)
- net AIN2: no longer U2.22 (AIN2)
- net Yellow: now reaches C1.1, RV1.2, U1.6 (IO34)
- new net: R1.1, U1.16 (IO13)
- new net IO12: U2.15 (PWMB)
- new net IO14: U2.16 (BIN2)
- new net IO25: U2.21 (AIN1)
- new net IO27: U2.17 (BIN1)
- new net IO32: U2.23 (PWMA)
- new net IO33: U2.22 (AIN2)
- new net PWMA: U1.8 (IO32)
- new net PWMB: U1.14 (IO12)
- new net STBY: U1.11 (IO26)
- no-connect marks 0 -> 29
Other:
- moved on the sheet: C1, D1, M1, M2, RV1, U1, U2

Commit message: Refactor hardware schematics: update GPIO assignments and add power flag symbols
Connections:
- net IO12 is gone; now on net PWMB: U2.15 (PWMB)
- net IO14 is gone; now on net BIN2: U2.16 (BIN2)
- net IO25 is gone; now on net AIN1: U2.21 (AIN1)
- net IO26 is gone; now on net STBY: U2.19 (STBY)
- net IO27 is gone; now on net BIN1: U2.17 (BIN1)
- net IO32 is gone; now on net PWMA: U2.23 (PWMA)
- net IO33 is gone; now on net AIN2: U2.22 (AIN2)
